Commit message: gogoo

File: src/fedar/robots/fedar.URDF (robot description, URDF)
Before this commit: robot fedar, 12 links, 11 joints
Joints:
- joint camera_joint: origin xyz=-0.25453 -0.05 1.204 rpy=0 0 -1.5708 -> xyz=-0.25453 -0.15 1.204 rpy=0 0.7 -1.5708
- joint lower_arm_joint: limit lower=0.1198 upper=1.6 effort=0 velocity=0 -> lower=-0.406 upper=0.320 effort=0 velocity=0
- joint upper_arm_joint: axis 0 0 1 -> 0 0 -1; limit lower=-0.05 upper=1.435 effort=0 velocity=0 -> lower=-0.051 upper=0.983 effort=0 velocity=0; origin xyz=0 0.015 0.9915 rpy=1.5708 -0.94746 -1.5708 -> xyz=0 0.015 0.9915 rpy=1.5708 -1.11746 -1.5708
